Commit message: [feat] update
Signed-off-by: duyongquan3 <duyongquan3@jd.com>

File: autonomy_ros/urdf/gz_waffle.sdf.xacro (robot description, xacro)
@@ -3,7 +3,12 @@
     <xacro:include filename="realsense_d435i_gz.xacro"/>
     <xacro:arg name="namespace" default=""/>
-    <model name="turtlebot3_waffle">
+    <xacro:arg name="robot_name" default="turtlebot3_waffle"/>
+    <!-- Absolute path to mesh directory (Gazebo Sim does not resolve package://). -->
+    <xacro:arg name="meshes_dir" default=""/>
+    <model name="$(arg robot_name)">
       <pose>0.0 0.0 0.0 0.0 0.0 0.0</pose>
-      <link name="base_footprint"/>
+      <link name="base_footprint">
+        <canonical_link/>
+      </link>
       <link name="base_link">
         <inertial>
@@ -31,5 +36,5 @@
           <geometry>
             <mesh>
-              <uri>package://autonomy_ros/models/turtlebot3_model/meshes/waffle_base.dae</uri>
+              <uri>file://$(arg meshes_dir)/waffle_base.dae</uri>
               <scale>0.001 0.001 0.001</scale>
             </mesh>
@@ -116,5 +121,5 @@
           <geometry>
             <mesh>
-              <uri>package://autonomy_ros/models/turtlebot3_model/meshes/lds.dae</uri>
+              <uri>file://$(arg meshes_dir)/lds.dae</uri>
               <scale>0.001 0.001 0.001</scale>
             </mesh>
@@ -190,5 +195,5 @@
                 <kp>1e+5</kp>
                 <kd>1</kd>
-                <max_vel>0.01</max_vel>
+                <max_vel>1.0</max_vel>
                 <min_depth>0.001</min_depth>
               </ode>
@@ -200,5 +205,5 @@
           <geometry>
             <mesh>
-              <uri>package://autonomy_ros/models/turtlebot3_model/meshes/tire.dae</uri>
+              <uri>file://$(arg meshes_dir)/tire.dae</uri>
               <scale>0.001 0.001 0.001</scale>
             </mesh>
@@ -240,4 +245,49 @@
               </ode>
             </friction>
+            <contact>
+              <ode>
+                <soft_cfm>0</soft_cfm>
+                <soft_erp>0.2</soft_erp>
+                <kp>1e+5</kp>
+                <kd>1</kd>
+                <max_vel>1.0</max_vel>
+                <min_depth>0.001</min_depth>
+              </ode>
+            </contact>
+          </surface>
+        </collision>
+        <visual name="wheel_right_visual">
+          <pose>0.0 -0.144 0.023 0 0 0</pose>
+          <geometry>
+            <mesh>
+              <uri>file://$(arg meshes_dir)/tire.dae</uri>
+              <scale>0.001 0.001 0.001</scale>
+            </mesh>
+          </geometry>
+          <material>
+            <diffuse>1 1 1</diffuse>
+          </material>
+        </visual>
+      </link>
+      <link name='caster_back_right_link'>
+        <pose>-0.177 -0.064 -0.004 0 0 0</pose>
+        <inertial>
+          <mass>0.001</mass>
+          <inertia>
+            <ixx>0.00001</ixx>
+            <ixy>0.000</ixy>
+            <ixz>0.000</ixz>
+            <iyy>0.00001</iyy>
+            <iyz>0.000</iyz>
+            <izz>0.00001</izz>
+          </inertia>
+        </inertial>
+        <collision name='collision'>
+          <geometry>
+            <sphere>
+              <radius>0.006000</radius>
+            </sphere>
+          </geometry>
+          <surface>
             <contact>
               <ode>
@@ -252,19 +302,7 @@
           </surface>
         </collision>
-        <visual name="wheel_right_visual">
-          <pose>0.0 -0.144 0.023 0 0 0</pose>
-          <geometry>
-            <mesh>
-              <uri>package://autonomy_ros/models/turtlebot3_model/meshes/tire.dae</uri>
-              <scale>0.001 0.001 0.001</scale>
-            </mesh>
-          </geometry>
-          <material>
-            <diffuse>1 1 1</diffuse>
-          </material>
-        </visual>
-      </link>
-      <link name='caster_back_right_link'>
-        <pose>-0.177 -0.064 -0.004 0 0 0</pose>
+      </link>
+      <link name='caster_back_left_link'>
+        <pose>-0.177 0.064 -0.004 0 0 0</pose>
         <inertial>
           <mass>0.001</mass>
@@ -298,40 +336,8 @@
         </collision>
       </link>
-      <link name='caster_back_left_link'>
-        <pose>-0.177 0.064 -0.004 0 0 0</pose>
-        <inertial>
-          <mass>0.001</mass>
-          <inertia>
-            <ixx>0.00001</ixx>
-            <ixy>0.000</ixy>
-            <ixz>0.000</ixz>
-            <iyy>0.00001</iyy>
-            <iyz>0.000</iyz>
-            <izz>0.00001</izz>
-          </inertia>
-        </inertial>
-        <collision name='collision'>
-          <geometry>
-            <sphere>
-              <radius>0.006000</radius>
-            </sphere>
-          </geometry>
-          <surface>
-            <contact>
-              <ode>
-                <soft_cfm>0</soft_cfm>
-                <soft_erp>0.2</soft_erp>
-                <kp>1e+5</kp>
-                <kd>1</kd>
-                <max_vel>0.01</max_vel>
-                <min_depth>0.001</min_depth>
-              </ode>
-            </contact>
-          </surface>
-        </collision>
-      </link>
+      <!-- camera_link origin is at camera_joint (front of base_link, +X forward). -->
       <link name="camera_link">
         <inertial>
-          <pose>0.069 -0.047 0.107 0 0 0</pose>
+          <pose>0 0 0 0 0 0</pose>
           <inertia>
             <ixx>0.001</ixx>
@@ -347,5 +353,5 @@
           <pose>0 0 0 0 0 0</pose>
           <geometry>
-            <!-- RealSense D435i body ~90 x 25 x 25 mm -->
+            <!-- RealSense D435i body ~90 x 25 x 25 mm (long axis along +X) -->
             <box>
               <size>0.090 0.025 0.025</size>
@@ -365,5 +371,7 @@
           </material>
         </visual>
-        <pose>0.069 -0.047 0.107 0 0 0</pose>
+      </link>
+      <link name="camera_color_frame"/>
+      <link name="camera_color_optical_frame">
         <xacro:realsense_d435i_sensor namespace="$(arg namespace)"/>
       </link>
@@ -412,4 +420,14 @@
           <xyz>0 0 1</xyz>
         </axis>
+      </joint>
+      <joint name="camera_color_joint" type="fixed">
+        <parent>camera_link</parent>
+        <child>camera_color_frame</child>
+        <pose>0 0 0 0 0 0</pose>
+      </joint>
+      <joint name="camera_color_optical_joint" type="fixed">
+        <parent>camera_color_frame</parent>
+        <child>camera_color_optical_frame</child>
+        <pose>0 0 0 -1.5708 0 -1.5708</pose>
       </joint>
       <joint name="imu_joint" type="fixed">
@@ -433,5 +451,5 @@
         <max_angular_velocity>1.9</max_angular_velocity>
         <min_angular_velocity>-1.9</min_angular_velocity>
-        <topic>$(arg namespace)/cmd_vel</topic>
+        <topic>/model/$(arg robot_name)/cmd_vel</topic>
         <odom_topic>$(arg namespace)/odom</odom_topic>
         <tf_topic>$(arg namespace)/tf</tf_topic>

File: autonomy_ros/urdf/realsense_d435i_gz.xacro (robot description, xacro)
@@ -9,4 +9,6 @@
       <visualize>false</visualize>
       <topic>${namespace}camera</topic>
+      <!-- Gazebo renders along sensor +X; align with ROS optical +Z. -->
+      <pose>0 0 0 1.5708 0 0</pose>
       <gz_frame_id>camera_color_optical_frame</gz_frame_id>
       <camera name="realsense_d435i">

Commit message: [feat] update
Signed-off-by: duyongquan3 <duyongquan3@jd.com>

File: autonomy_ros/urdf/gz_waffle.sdf.xacro (robot description, xacro)
@@ -1,26 +1,23 @@
 <?xml version="1.0"?>
 <sdf version="1.6" xmlns:xacro="http://www.ros.org/wiki/xacro">
-    <xacro:include filename="realsense_d435i_gz.xacro"/>
     <xacro:arg name="namespace" default=""/>
     <xacro:arg name="robot_name" default="turtlebot3_waffle"/>
-    <!-- Absolute path to mesh directory (Gazebo Sim does not resolve package://). -->
+    <!-- Gazebo Sim does not resolve package://; pass absolute meshes_dir from launch. -->
     <xacro:arg name="meshes_dir" default=""/>
     <model name="$(arg robot_name)">
       <pose>0.0 0.0 0.0 0.0 0.0 0.0</pose>
-      <link name="base_footprint">
-        <canonical_link/>
-      </link>
+      <link name="base_footprint"/>
       <link name="base_link">
         <inertial>
           <pose>-0.064 0 0.048 0 0 0</pose>
           <inertia>
-            <ixx>0.001</ixx>
-            <ixy>0.000</ixy>
-            <ixz>0.000</ixz>
-            <iyy>0.001</iyy>
-            <iyz>0.000</iyz>
-            <izz>0.001</izz>
-          </inertia>
-          <mass>1.0</mass>
+            <ixx>4.2111447e-02</ixx>
+            <ixy>0</ixy>
+            <ixz>0</ixz>
+            <iyy>4.2111447e-02</iyy>
+            <iyz>0</iyz>
+            <izz>7.5254874e-02</izz>
+          </inertia>
+          <mass>1.3729096</mass>
         </inertial>
         <collision name="base_collision">
@@ -97,5 +94,5 @@
       <link name="base_scan">
         <inertial>
-          <pose>-0.064 0 0.121 0 0 0</pose>
+          <pose>-0.052 0 0.111 0 0 0</pose>
           <inertia>
             <ixx>0.001</ixx>
@@ -106,5 +103,5 @@
             <izz>0.001</izz>
           </inertia>
-          <mass>0.125</mass>
+          <mass>0.114</mass>
         </inertial>
         <collision name="lidar_sensor_collision">
@@ -161,13 +158,13 @@
         <inertial>
           <pose>0.0 0.144 0.023 -1.57 0 0</pose>
-          <inertia>
-            <ixx>0.001</ixx>
-            <ixy>0.000</ixy>
-            <ixz>0.000</ixz>
-            <iyy>0.001</iyy>
-            <iyz>0.000</iyz>
-            <izz>0.001</izz>
-          </inertia>
           <mass>0.1</mass>
+          <inertia>
+            <ixx>1.1175580e-05</ixx>
+            <ixy>0.0</ixy>
+            <ixz>0.0</ixz>
+            <iyy>1.1192413e-05</iyy>
+            <iyz>0.0</iyz>
+            <izz>2.0712558e-05</izz>
+          </inertia>
         </inertial>
         <collision name="wheel_left_collision">
@@ -182,9 +179,9 @@
             <friction>
               <ode>
-                <mu>1</mu>
-                <mu2>1</mu2>
-                <slip1>0.035</slip1>
-                <slip2>0</slip2>
+                <mu>100000.0</mu>
+                <mu2>100000.0</mu2>
                 <fdir1>0 0 1</fdir1>
+                <slip1>0.0</slip1>
+                <slip2>0.0</slip2>
               </ode>
             </friction>
@@ -195,5 +192,5 @@
                 <kp>1e+5</kp>
                 <kd>1</kd>
-                <max_vel>1.0</max_vel>
+                <max_vel>0.01</max_vel>
                 <min_depth>0.001</min_depth>
               </ode>
@@ -217,13 +214,13 @@
         <inertial>
           <pose>0.0 -0.144 0.023 -1.57 0 0</pose>
-          <inertia>
-            <ixx>0.001</ixx>
-            <ixy>0.000</ixy>
-            <ixz>0.000</ixz>
-            <iyy>0.001</iyy>
-            <iyz>0.000</iyz>
-            <izz>0.001</izz>
-          </inertia>
           <mass>0.1</mass>
+          <inertia>
+            <ixx>1.1175580e-05</ixx>
+            <ixy>0.0</ixy>
+            <ixz>0.0</ixz>
+            <iyy>1.1192413e-05</iyy>
+            <iyz>0.0</iyz>
+            <izz>2.0712558e-05</izz>
+          </inertia>
         </inertial>
         <collision name="wheel_right_collision">
@@ -238,9 +235,9 @@
             <friction>
               <ode>
-                <mu>1</mu>
-                <mu2>1</mu2>
-                <slip1>0.035</slip1>
-                <slip2>0</slip2>
+                <mu>100000.0</mu>
+                <mu2>100000.0</mu2>
                 <fdir1>0 0 1</fdir1>
+                <slip1>0.0</slip1>
+                <slip2>0.0</slip2>
               </ode>
             </friction>
@@ -251,5 +248,5 @@
                 <kp>1e+5</kp>
                 <kd>1</kd>
-                <max_vel>1.0</max_vel>
+                <max_vel>0.01</max_vel>
                 <min_depth>0.001</min_depth>
               </ode>
@@ -270,5 +267,5 @@
         </visual>
       </link>
-      <link name='caster_back_right_link'>
+      <link name="caster_back_right_link">
         <pose>-0.177 -0.064 -0.004 0 0 0</pose>
         <inertial>
@@ -283,8 +280,8 @@
           </inertia>
         </inertial>
-        <collision name='collision'>
+        <collision name="collision">
           <geometry>
             <sphere>
-              <radius>0.006000</radius>
+              <radius>0.006</radius>
             </sphere>
           </geometry>
@@ -303,5 +300,5 @@
         </collision>
       </link>
-      <link name='caster_back_left_link'>
+      <link name="caster_back_left_link">
         <pose>-0.177 0.064 -0.004 0 0 0</pose>
         <inertial>
@@ -316,8 +313,8 @@
           </inertia>
         </inertial>
-        <collision name='collision'>
+        <collision name="collision">
           <geometry>
             <sphere>
-              <radius>0.006000</radius>
+              <radius>0.006</radius>
             </sphere>
           </geometry>
@@ -336,44 +333,4 @@
         </collision>
       </link>
-      <!-- camera_link origin is at camera_joint (front of base_link, +X forward). -->
-      <link name="camera_link">
-        <inertial>
-          <pose>0 0 0 0 0 0</pose>
-          <inertia>
-            <ixx>0.001</ixx>
-            <ixy>0.000</ixy>
-            <ixz>0.000</ixz>
-            <iyy>0.001</iyy>
-            <iyz>0.000</iyz>
-            <izz>0.001</izz>
-          </inertia>
-          <mass>0.072</mass>
-        </inertial>
-        <collision name="collision">
-          <pose>0 0 0 0 0 0</pose>
-          <geometry>
-            <!-- RealSense D435i body ~90 x 25 x 25 mm (long axis along +X) -->
-            <box>
-              <size>0.090 0.025 0.025</size>
-            </box>
-          </geometry>
-        </collision>
-        <visual name="realsense_d435i_visual">
-          <pose>0 0 0 0 0 0</pose>
-          <geometry>
-            <box>
-              <size>0.090 0.025 0.025</size>
-            </box>
-          </geometry>
-          <material>
-            <ambient>0.2 0.2 0.2 1</ambient>
-            <diffuse>0.3 0.3 0.35 1</diffuse>
-          </material>
-        </visual>
-      </link>
-      <link name="camera_color_frame"/>
-      <link name="camera_color_optical_frame">
-        <xacro:realsense_d435i_sensor namespace="$(arg namespace)"/>
-      </link>
       <joint name="base_joint" type="fixed">
         <parent>base_footprint</parent>
@@ -397,9 +354,9 @@
         </axis>
       </joint>
-      <joint name='caster_back_right_joint' type='ball'>
+      <joint name="caster_back_right_joint" type="ball">
         <parent>base_link</parent>
         <child>caster_back_right_link</child>
       </joint>
-      <joint name='caster_back_left_joint' type='ball'>
+      <joint name="caster_back_left_joint" type="ball">
         <parent>base_link</parent>
         <child>caster_back_left_link</child>
@@ -409,25 +366,4 @@
         <child>base_scan</child>
         <pose>-0.064 0 0.121 0 0 0</pose>
-        <axis>
-          <xyz>0 0 1</xyz>
-        </axis>
-      </joint>
-      <joint name="camera_joint" type="fixed">
-        <parent>base_link</parent>
-        <child>camera_link</child>
-        <pose>0.064 -0.065 0.094 0 0 0</pose>
-        <axis>
-          <xyz>0 0 1</xyz>
-        </axis>
-      </joint>
-      <joint name="camera_color_joint" type="fixed">
-        <parent>camera_link</parent>
-        <child>camera_color_frame</child>
-        <pose>0 0 0 0 0 0</pose>
-      </joint>
-      <joint name="camera_color_optical_joint" type="fixed">
-        <parent>camera_color_frame</parent>
-        <child>camera_color_optical_frame</child>
-        <pose>0 0 0 -1.5708 0 -1.5708</pose>
       </joint>
       <joint name="imu_joint" type="fixed">

File: autonomy_ros/urdf/gz_waffle_gps.sdf.xacro (robot description, xacro)
@@ -376,53 +376,4 @@
         </visual>
       </link>
-      <link name="camera_link">
-        <inertial>
-          <pose>0.069 -0.047 0.107 0 0 0</pose>
-          <inertia>
-            <ixx>0.001</ixx>
-            <ixy>0.000</ixy>
-            <ixz>0.000</ixz>
-            <iyy>0.001</iyy>
-            <iyz>0.000</iyz>
-            <izz>0.001</izz>
-          </inertia>
-          <mass>0.035</mass>
-        </inertial>
-        <collision name="collision">
-          <pose>0 0.047 -0.005 0 0 0</pose>
-          <geometry>
-            <box>
-              <size>0.008 0.130 0.022</size>
-            </box>
-          </geometry>
-        </collision>
-        <pose>0.069 -0.047 0.107 0 0 0</pose>
-        <sensor name="intel_realsense_r200_depth" type="depth">
-          <always_on>1</always_on>
-          <update_rate>5</update_rate>
-          <pose>0.064 -0.047 0.107 0 0 0</pose>
-          <gz_frame_id>camera_depth_frame</gz_frame_id>
-          <camera name="realsense_depth_camera">
-            <horizontal_fov>1.047</horizontal_fov>
-            <image>
-              <width>320</width>
-              <height>240</height>
-            </image>
-            <lens>
-              <projection>
-                <!-- focal_length = fx = fy = width / ( 2 * tan (hfov / 2 ) ) -->
-                <!-- tx = hackBaseline * focal_length -->
-                <tx>19.4</tx>
-              </projection>
-            </lens>
-            <depth_camera>
-              <clip>
-                <near>0.001</near>
-                <far>5.0</far>
-              </clip>
-            </depth_camera>
-          </camera>
-        </sensor>
-      </link>
       <joint name="base_joint" type="fixed">
         <parent>base_footprint</parent>
@@ -458,12 +409,4 @@
         <child>base_scan</child>
         <pose>-0.064 0 0.121 0 0 0</pose>
-        <axis>
-          <xyz>0 0 1</xyz>
-        </axis>
-      </joint>
-      <joint name="camera_joint" type="fixed">
-        <parent>base_link</parent>
-        <child>camera_link</child>
-        <pose>0.064 -0.065 0.094 0 0 0</pose>
         <axis>
           <xyz>0 0 1</xyz>

File: autonomy_ros/urdf/turtlebot3_waffle.urdf (robot description, URDF)
Before this commit: robot turtlebot3_waffle, 13 links, 12 joints
Links:
- removed link camera_color_frame
- removed link camera_color_optical_frame
- removed link camera_depth_frame
- removed link camera_depth_optical_frame
- removed link camera_link
Joints:
- removed joint camera_color_joint
- removed joint camera_color_optical_joint
- removed joint camera_depth_joint
- removed joint camera_depth_optical_joint
- removed joint camera_joint

File: autonomy_ros/urdf/turtlebot3_waffle_gps.urdf (robot description, URDF)
Before this commit: robot turtlebot3_waffle, 14 links, 13 joints
Links:
- removed link camera_depth_frame
- removed link camera_depth_optical_frame
- removed link camera_link
- removed link camera_rgb_frame
- removed link camera_rgb_optical_frame
Joints:
- removed joint camera_depth_joint
- removed joint camera_depth_optical_joint
- removed joint camera_joint
- removed joint camera_rgb_joint
- removed joint camera_rgb_optical_joint

File: autonomy_ros/worlds/tb3_sandbox.sdf.xacro (robot description, xacro)
@@ -72,4 +72,10 @@
         <max_step_size>0.003</max_step_size>
         <real_time_factor>1</real_time_factor>
+        <ode>
+          <solver>
+            <iters>50</iters>
+            <sor>1.3</sor>
+          </solver>
+        </ode>
     </physics>
     <model name="turtlebot3_world">
