Commit message: update

File: autonomy_simulator/urdf/gz_waffle_gps.sdf.xacro (robot description, xacro)
@@ -30,5 +30,5 @@
           <geometry>
             <mesh>
-              <uri>package://autonomy_ros/models/turtlebot3_model/meshes/waffle_base.dae</uri>
+              <uri>package://autonomy_simulator/models/turtlebot3_model/meshes/waffle_base.dae</uri>
               <scale>0.001 0.001 0.001</scale>
             </mesh>
@@ -141,5 +141,5 @@
           <geometry>
             <mesh>
-              <uri>package://autonomy_ros/models/turtlebot3_model/meshes/lds.dae</uri>
+              <uri>package://autonomy_simulator/models/turtlebot3_model/meshes/lds.dae</uri>
               <scale>0.001 0.001 0.001</scale>
             </mesh>
@@ -225,5 +225,5 @@
           <geometry>
             <mesh>
-              <uri>package://autonomy_ros/models/turtlebot3_model/meshes/tire.dae</uri>
+              <uri>package://autonomy_simulator/models/turtlebot3_model/meshes/tire.dae</uri>
               <scale>0.001 0.001 0.001</scale>
             </mesh>
@@ -281,5 +281,5 @@
           <geometry>
             <mesh>
-              <uri>package://autonomy_ros/models/turtlebot3_model/meshes/tire.dae</uri>
+              <uri>package://autonomy_simulator/models/turtlebot3_model/meshes/tire.dae</uri>
               <scale>0.001 0.001 0.001</scale>
             </mesh>

File: autonomy_simulator/urdf/turtlebot3_waffle.urdf (robot description, URDF)
Before this commit: robot turtlebot3_waffle, 8 links, 7 joints
Links:
- link base_link: geometry collision box size=0.266 0.266 0.094; visual mesh filename=package://autonomy_simulator/models/turtlebot3_model/meshes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 scale=0.001 0.001 0.001
- link base_scan: geometry collision cylinder length=0.0315 radius=0.055; visual mesh filename=package://autonomy_simulator/models/turtlebot3_model/meshes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 scale=0.001 0.001 0.001
- link wheel_left_link: geometry collision cylinder length=0.018 radius=0.033; visual mesh filename=package://autonomy_simulator/models/turtlebot3_model/meshes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 scale=0.001 0.001 0.001
- link wheel_right_link: geometry collision cylinder length=0.018 radius=0.033; visual mesh filename=package://autonomy_simulator/models/turtlebot3_model/meshes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 scale=0.001 0.001 0.001

File: autonomy_simulator/urdf/turtlebot3_waffle_gps.urdf (robot description, URDF)
Before this commit: robot turtlebot3_waffle, 9 links, 8 joints
Links:
- link base_link: geometry collision box size=0.266 0.266 0.094; visual mesh filename=package://autonomy_simulator/models/turtlebot3_model/meshes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 scale=0.001 0.001 0.001
- link base_scan: geometry collision cylinder length=0.0315 radius=0.055; visual mesh filename=package://autonomy_simulator/models/turtlebot3_model/meshes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 scale=0.001 0.001 0.001
- link wheel_left_link: geometry collision cylinder length=0.018 radius=0.033; visual mesh filename=package://autonomy_simulator/models/turtlebot3_model/meshes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 scale=0.001 0.001 0.001
- link wheel_right_link: geometry collision cylinder length=0.018 radius=0.033; visual mesh filename=package://autonomy_simulator/models/turtlebot3_model/meshes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 scale=0.001 0.001 0.001
